File: pcb/_autosave-pcb.kicad_sch (KiCad schematic)
At the start: 11 parts, among them J1 Conn_01x15 Right, J2 Conn_01x15 Left, P1 Conn_01x06, U1 STM32F756VGTx, U2 MP34DT05-A, U3 ISM330DHCX

Commit message: pcb_4
Parts:
- added J3: DIN41612_02x08_AB_EvenPins, Connector_PinSocket_2.54mm:PinSocket_2x08_P2.54mm_Horizontal, symbol Connector:DIN41612_02x08_AB_EvenPins
Connections:
- net GND: now also J3.b2 (Pin_b2)
- net VDD: now also J3.a2 (Pin_a2)
- net SAI1_FS: now reaches U1.3 (PE4)
- net SAI1_FS: now also J3.b16 (Pin_b16)
- net SPI3_MOSI: now reaches U1.36 (PB2)
- net SPI3_MOSI: now also J3.b6 (Pin_b6)
- net SAI1_SCK: now reaches U1.4 (PE5)
- net SAI1_SCK: now also J3.b14 (Pin_b14)
- net SPI4_NSS: now reaches U1.41 (PE11)
- net SPI4_NSS: now also J3.a10 (Pin_a10)
- net SPI4_SCK: now reaches U1.42 (PE12)
- net SPI4_SCK: now also J3.a8 (Pin_a8)
- net SPI4_MISO: now reaches U1.43 (PE13)
- net SPI4_MISO: now also J3.a4 (Pin_a4)
- net SPI4_MOSI: now reaches U1.44 (PE14)
- net SPI4_MOSI: now also J3.a6 (Pin_a6)
- net SAI2_SD: now reaches U1.58 (PD11)
- net SAI2_SD: now also J3.a12 (Pin_a12)
- net SAI2_FS: now reaches U1.59 (PD12)
- net SAI2_FS: now also J3.a16 (Pin_a16)
- net SAI2_SCK: now reaches U1.60 (PD13)
- net SAI2_SCK: now also J3.a14 (Pin_a14)
- net SPI3_NSS: now reaches U1.77 (PA15)
- net SPI3_NSS: now also J3.b10 (Pin_b10)
- net SPI3_SCK: now reaches U1.78 (PC10)
- net SPI3_SCK: now also J3.b8 (Pin_b8)
- net SPI3_MISO: now reaches U1.79 (PC11)
- net SPI3_MISO: now also J3.b4 (Pin_b4)
- net SAI1_SD: now reaches U1.87 (PD6)
- net SAI1_SD: now also J3.b12 (Pin_b12)
Changed lines of the file:
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@@
+    (stroke (width 0) (type default) (color 0 0 0 0))
+  )
+  (wire (pts (xy 138.43 138.43) (xy 127 138.43))
     (stroke (width 0) (type default) (color 0 0 0 0))
   )
@@
   )
   (wire (pts (xy 133.35 96.52) (xy 133.35 97.79))
+    (stroke (width 0) (type default) (color 0 0 0 0))
+  )
+  (wire (pts (xy 102.87 138.43) (xy 114.3 138.43))
     (stroke (width 0) (type default) (color 0 0 0 0))
   )
@@
     (effects (font (size 1.27 1.27)) (justify right bottom))
   )
+  (label "SAI2_SD" (at 114.3 151.13 180)
+    (effects (font (size 1.27 1.27)) (justify right bottom))
+  )
   (label "SPI1_SCK" (at 245.11 80.01 180)
     (effects (font (size 1.27 1.27)) (justify right bottom))
   )
+  (label "SPI4_SCK" (at 114.3 146.05 180)
+    (effects (font (size 1.27 1.27)) (justify right bottom))
+  )
   (label "SWDIO" (at 71.12 76.2 0)
     (effects (font (size 1.27 1.27)) (justify left bottom))
   )
+  (label "SPI4_MOSI" (at 114.3 143.51 180)
+    (effects (font (size 1.27 1.27)) (justify right bottom))
+  )
+  (label "SPI4_MISO" (at 27.94 119.38 180)
+    (effects (font (size 1.27 1.27)) (justify right bottom))
+  )
+  (label "SPI4_NSS" (at 27.94 114.3 180)
+    (effects (font (size 1.27 1.27)) (justify right bottom))
+  )
   (label "SPI1_MISO" (at 245.11 82.55 180)
     (effects (font (size 1.27 1.27)) (justify right bottom))
   )
+  (label "SPI3_SCK" (at 71.12 154.94 0)
+    (effects (font (size 1.27 1.27)) (justify left bottom))
+  )
+  (label "SPI3_MOSI" (at 71.12 91.44 0)
+    (effects (font (size 1.27 1.27)) (justify left bottom))
+  )
+  (label "SPI3_NSS" (at 71.12 81.28 0)
+    (effects (font (size 1.27 1.27)) (justify left bottom))
+  )
+  (label "SAI1_SCK" (at 127 153.67 0)
+    (effects (font (size 1.27 1.27)) (justify left bottom))
+  )
+  (label "SPI3_SCK" (at 127 146.05 0)
+    (effects (font (size 1.27 1.27)) (justify left bottom))
+  )
+  (label "SPI4_SCK" (at 27.94 116.84 180)
+    (effects (font (size 1.27 1.27)) (justify right bottom))
+  )
   (label "NRST" (at 252.73 21.59 180)
     (effects (font (size 1.27 1.27)) (justify right bottom))
@@
     (effects (font (size 1.27 1.27)) (justify left bottom))
   )
+  (label "SAI2_FS" (at 27.94 160.02 180)
+    (effects (font (size 1.27 1.27)) (justify right bottom))
+  )
+  (label "SPI3_MISO" (at 71.12 157.48 0)
+    (effects (font (size 1.27 1.27)) (justify left bottom))
+  )
   (label "SWO" (at 252.73 24.13 180)
     (effects (font (size 1.27 1.27)) (justify right bottom))
   )
+  (label "SAI2_SD" (at 27.94 157.48 180)
+    (effects (font (size 1.27 1.27)) (justify right bottom))
+  )
   (label "SWO" (at 71.12 93.98 0)
     (effects (font (size 1.27 1.27)) (justify left bottom))
@@
     (effects (font (size 1.27 1.27)) (justify right bottom))
   )
+  (label "SPI3_MISO" (at 127 140.97 0)
+    (effects (font (size 1.27 1.27)) (justify left bottom))
+  )
   (label "SPI1_MISO" (at 71.12 58.42 0)
     (effects (font (size 1.27 1.27)) (justify left bottom))
@@
     (effects (font (size 1.27 1.27)) (justify left bottom))
   )
+  (label "SAI1_FS" (at 127 156.21 0)
+    (effects (font (size 1.27 1.27)) (justify left bottom))
+  )
   (label "SPI2_CLK" (at 71.12 66.04 0)
     (effects (font (size 1.27 1.27)) (justify left bottom))
   )
+  (label "SAI2_SCK" (at 27.94 162.56 180)
+    (effects (font (size 1.27 1.27)) (justify right bottom))
+  )
+  (label "SAI2_SCK" (at 114.3 153.67 180)
+    (effects (font (size 1.27 1.27)) (justify right bottom))
+  )
   (label "I2C1_SCL" (at 71.12 101.6 0)
     (effects (font (size 1.27 1.27)) (justify left bottom))
@@
     (effects (font (size 1.27 1.27)) (justify right bottom))
   )
+  (label "SPI3_NSS" (at 127 148.59 0)
+    (effects (font (size 1.27 1.27)) (justify left bottom))
+  )
   (label "SWCLK" (at 71.12 78.74 0)
     (effects (font (size 1.27 1.27)) (justify left bottom))
   )
+  (label "SAI1_SD" (at 127 151.13 0)
+    (effects (font (size 1.27 1.27)) (justify left bottom))
+  )
+  (label "SPI4_MOSI" (at 27.94 121.92 180)
+    (effects (font (size 1.27 1.27)) (justify right bottom))
+  )
   (label "SPI1_MOSI" (at 71.12 60.96 0)
     (effects (font (size 1.27 1.27)) (justify left bottom))
@@
     (effects (font (size 1.27 1.27)) (justify right bottom))
   )
+  (label "SAI1_SCK" (at 27.94 99.06 180)
+    (effects (font (size 1.27 1.27)) (justify right bottom))
+  )
+  (label "SPI4_NSS" (at 114.3 148.59 180)
+    (effects (font (size 1.27 1.27)) (justify right bottom))
+  )
+  (label "SAI1_FS" (at 27.94 96.52 180)
+    (effects (font (size 1.27 1.27)) (justify right bottom))
+  )
+  (label "SPI4_MISO" (at 114.3 140.97 180)
+    (effects (font (size 1.27 1.27)) (justify right bottom))
+  )
+  (label "SAI1_SD" (at 27.94 144.78 180)
+    (effects (font (size 1.27 1.27)) (justify right bottom))
+  )
   (label "SPI2_MISO" (at 71.12 134.62 0)
+    (effects (font (size 1.27 1.27)) (justify left bottom))
+  )
+  (label "SAI2_FS" (at 114.3 156.21 180)
+    (effects (font (size 1.27 1.27)) (justify right bottom))
+  )
+  (label "SPI3_MOSI" (at 127 143.51 0)
     (effects (font (size 1.27 1.27)) (justify left bottom))
   )
@@
     (pin "99")
   )
+  (symbol (lib_id "Connector:DIN41612_02x08_AB_EvenPins") (at 119.38 146.05 0) (unit 1)
+    (in_bom yes) (on_board yes) (fields_autoplaced)
+    (property "Reference" "J3" (id 0) (at 120.65 132.08 0))
+    (property "Value" "DIN41612_02x08_AB_EvenPins" (id 1) (at 120.65 134.62 0))
+    (property "Footprint" "Connector_PinSocket_2.54mm:PinSocket_2x08_P2.54mm_Horizontal" (id 2) (at 119.38 146.05 0)
+      (effects (font (size 1.27 1.27)) hide)
+    )
+    (property "Datasheet" "~" (id 3) (at 119.38 146.05 0)
+      (effects (font (size 1.27 1.27)) hide)
+    )
+    (pin "a10")
+    (pin "a12")
+    (pin "a14")
+    (pin "a16")
+    (pin "a2")
+    (pin "a4")
+    (pin "a6")
+    (pin "a8")
+    (pin "b10")
+    (pin "b12")
+    (pin "b14")
+    (pin "b16")
+    (pin "b2")
+    (pin "b4")
+    (pin "b6")
+    (pin "b8")
+  )
   (symbol (lib_id "Device:R") (at 175.26 68.58 90) (unit 1)
     (in_bom yes) (on_board yes) (fields_autoplaced)
@@
     (pin "6")
   )
+  (symbol (lib_id "power:VDD") (at 102.87 138.43 90) (unit 1)
+    (in_bom yes) (on_board yes) (fields_autoplaced)
+    (property "Reference" "#PWR?" (id 0) (at 106.68 138.43 0)
+      (effects (font (size 1.27 1.27)) hide)
+    )
+    (property "Value" "VDD" (id 1) (at 99.06 138.4299 90)
+      (effects (font (size 1.27 1.27)) (justify left))
+    )
+    (property "Footprint" "" (id 2) (at 102.87 138.43 0)
+      (effects (font (size 1.27 1.27)) hide)
+    )
+    (property "Datasheet" "" (id 3) (at 102.87 138.43 0)
+      (effects (font (size 1.27 1.27)) hide)
+    )
+    (pin "1")
+  )
   (symbol (lib_id "power:VDD") (at 114.3 41.91 180) (unit 1)
     (in_bom yes) (on_board yes) (fields_autoplaced)
@@
     (pin "VDD")
   )
+  (symbol (lib_id "power:GND") (at 138.43 138.43 90) (unit 1)
+    (in_bom yes) (on_board yes) (fields_autoplaced)
+    (property "Reference" "#PWR?" (id 0) (at 144.78 138.43 0)
+      (effects (font (size 1.27 1.27)) hide)
+    )
+    (property "Value" "GND" (id 1) (at 142.24 138.4299 90)
+      (effects (font (size 1.27 1.27)) (justify right))
+    )
+    (property "Footprint" "" (id 2) (at 138.43 138.43 0)
+      (effects (font (size 1.27 1.27)) hide)
+    )
+    (property "Datasheet" "" (id 3) (at 138.43 138.43 0)
+      (effects (font (size 1.27 1.27)) hide)
+    )
+    (pin "1")
+  )
   (symbol (lib_id "power:GND") (at 227.33 77.47 270) (unit 1)
     (in_bom yes) (on_board yes) (fields_autoplaced)
@@
       (reference "#PWR?") (unit 1) (value "VDD") (footprint "")
     )
+    (path "/8c60e3c9-4275-4a7b-9593-0d6ad7af9d00"
+      (reference "#PWR?") (unit 1) (value "VDD") (footprint "")
+    )
     (path "/93d65058-5cec-4c35-8b06-3f31a92b18cb"
       (reference "#PWR?") (unit 1) (value "VDD") (footprint "")
@@
       (reference "#PWR?") (unit 1) (value "GND") (footprint "")
     )
+    (path "/cb86b11f-c4b7-46f0-a3c8-d7b8474868aa"
+      (reference "#PWR?") (unit 1) (value "GND") (footprint "")
+    )
     (path "/f741d2a6-3cfd-425c-b5b1-c8b6c7563112"
       (reference "#PWR?") (unit 1) (value "GND") (footprint "")
@@
       (reference "J2") (unit 1) (value "Conn_01x15 Left") (footprint "Connector_PinSocket_2.54mm:PinSocket_1x15_P2.54mm_Vertical")
     )
+    (path "/39704ed7-9bbe-4b0b-b956-2fe0a3bd7ddb"
+      (reference "J3") (unit 1) (value "DIN41612_02x08_AB_EvenPins") (footprint "Connector_PinSocket_2.54mm:PinSocket_2x08_P2.54mm_Horizontal")
+    )
     (path "/8a48b6fa-d742-44c7-b137-f06bed0efe74"
