File: pcb/pcb.kicad_pcb (KiCad board)
At the start: 2 copper layers, 2 parts, among them P1 Conn_01x06, U1 STM32F756VGTx

Commit message: pcb_6
Parts:
- added C1: 100nF, Capacitor_SMD:C_0201_0603Metric, B.Cu at (116.3, 126.3)
- added C2: 1uF, Resistor_SMD:R_0201_0603Metric, B.Cu at (113.1, 110.4)
- added C3: 100nF, Resistor_SMD:R_0201_0603Metric, B.Cu at (113.2, 111.5)
- added J1: Conn_01x15 Right, Connector_PinSocket_2.54mm:PinSocket_1x15_P2.54mm_Vertical, F.Cu at (99.1, 94.0)
- added J2: Conn_01x15 Left, Connector_PinSocket_2.54mm:PinSocket_1x15_P2.54mm_Vertical, F.Cu at (127.0, 94.0)
- added J3: DIN41612_02x08_AB_EvenPins, Connector_PinSocket_2.54mm:PinSocket_2x08_P2.54mm_Horizontal, B.Cu at (104.2, 105.4)
- added R1: 10kOhm, Resistor_SMD:R_0201_0603Metric, B.Cu at (108.2, 113.8)
- added R2: 10kOhm, Resistor_SMD:R_0201_0603Metric, B.Cu at (108.4, 119.6)
- added U2: MP34DT05-A, lol:MIC-PACK, B.Cu at (113.3, 113.7)
- added U3: ISM330DHCX, ISM:LGA-14L, B.Cu at (113.2, 119.8)
- moved P1 57.8 mm to (110.5, 129.5)
- moved U1 34.1 mm to (112.7, 116.5), turned to -90 degrees
Connections:
- U1 pad 17: unconnected-(U1-Pad17) -> /SPI2_MISO
- U1 pad 28: unconnected-(U1-Pad28) -> GND
- U1 pad 29: unconnected-(U1-Pad29) -> /SPI1_SCK
- U1 pad 3: unconnected-(U1-Pad3) -> /SAI1_FS
- U1 pad 30: unconnected-(U1-Pad30) -> /SPI1_MISO
- U1 pad 31: unconnected-(U1-Pad31) -> /SPI1_MOSI
- U1 pad 36: unconnected-(U1-Pad36) -> /SPI3_MOSI
- U1 pad 4: unconnected-(U1-Pad4) -> /SAI1_SCK
- U1 pad 41: unconnected-(U1-Pad41) -> /SPI4_NSS
- U1 pad 42: unconnected-(U1-Pad42) -> /SPI4_SCK
- U1 pad 43: unconnected-(U1-Pad43) -> /SPI4_MISO
- U1 pad 44: unconnected-(U1-Pad44) -> /SPI4_MOSI
- U1 pad 58: unconnected-(U1-Pad58) -> /SAI2_SD
- U1 pad 59: unconnected-(U1-Pad59) -> /SAI2_FS
- U1 pad 60: unconnected-(U1-Pad60) -> /SAI2_SCK
- U1 pad 68: unconnected-(U1-Pad68) -> /SPI2_CLK
- U1 pad 77: unconnected-(U1-Pad77) -> /SPI3_NSS
- U1 pad 78: unconnected-(U1-Pad78) -> /SPI3_SCK
- U1 pad 79: unconnected-(U1-Pad79) -> /SPI3_MISO
- U1 pad 87: unconnected-(U1-Pad87) -> /SAI1_SD
- U1 pad 92: unconnected-(U1-Pad92) -> /I2C1_SCL
- U1 pad 93: unconnected-(U1-Pad93) -> /I2C1_SDA
Routing:
- net VDD: track 0.00 -> 61.1 mm, vias 0 -> 6
- net GND: track 0.00 -> 60.6 mm, vias 0 -> 3
- net /NRST: track 0.00 -> 56.0 mm
- net /SPI3_MISO: track 0.00 -> 39.6 mm, vias 0 -> 3
- net /SPI4_SCK: track 0.00 -> 32.3 mm, vias 0 -> 2
- net /SPI3_NSS: track 0.00 -> 31.0 mm, vias 0 -> 1
- net /SAI2_FS: track 0.00 -> 26.8 mm, vias 0 -> 1
- net /SPI4_MOSI: track 0.00 -> 26.0 mm, vias 0 -> 1
- net /SPI3_SCK: track 0.00 -> 24.8 mm, vias 0 -> 3
- net /SWO: track 0.00 -> 24.7 mm, vias 0 -> 1
- net /SAI2_SCK: track 0.00 -> 24.0 mm, vias 0 -> 1
- net /SAI2_SD: track 0.00 -> 22.6 mm, vias 0 -> 1
- net /I2C1_SCL: track 0.00 -> 20.8 mm, vias 0 -> 2
- net /SPI4_NSS: track 0.00 -> 19.9 mm, vias 0 -> 2
- net /SPI1_MOSI: track 0.00 -> 17.2 mm
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- added copper zone on F.Cu, net GND
Other:
- board outline added: 33 x 40.6 mm

Commit message: pcb_8
Parts:
- added C4: 100nF, Capacitor_SMD:C_0201_0603Metric, F.Cu at (113.7, 128.9)
- added C5: 100nF, Capacitor_SMD:C_0201_0603Metric, F.Cu at (113.7, 130.2)
- added C6: 100nF, Capacitor_SMD:C_0201_0603Metric, F.Cu at (113.7, 131.4)
- added C7: 1pF, Capacitor_SMD:C_0201_0603Metric, F.Cu at (114.9, 120.7)
- added C8: 1pF, Capacitor_SMD:C_0201_0603Metric, F.Cu at (114.9, 111.8)
- added D1: LED, Diode_SMD:D_0201_0603Metric, B.Cu at (104.8, 118.1)
- added R3: 680ohm, Resistor_SMD:R_0201_0603Metric, B.Cu at (104.8, 119.7)
- added Y1: Crystal, Crystal:Crystal_SMD_Abracon_ABM3-2Pin_5.0x3.2mm, F.Cu at (114.9, 116.2)
- C1, C2, C3, R1, R2: moved to F.Cu
- moved C3 16.2 mm to (113.7, 127.6), turned to 0 degrees
- moved C2 15.9 mm to (113.7, 126.4), turned to 0 degrees
- moved R1 14.4 mm to (108.6, 128.3)
- moved J3 10.4 mm to (96.5, 98.3)
- moved U2 10.4 mm to (102.9, 113.7), turned to 0 degrees
- moved U1 9.20 mm to (103.5, 116.8), turned to 180 degrees
- moved U3 8.84 mm to (106.8, 113.7), turned to 0 degrees
- moved R2 8.83 mm to (109.9, 128.3)
- moved P1 8.59 mm to (102.3, 132.1)
- moved J2 8.04 mm to (119.4, 96.5)
- moved J1 8.02 mm to (91.5, 96.5)
- moved C1 2.88 mm to (113.7, 125.1), turned to 0 degrees
Connections:
- U1 pad 12: unconnected-(U1-Pad12) -> /OSC_IN
- U1 pad 13: unconnected-(U1-Pad13) -> /OSC_OUT
- U1 pad 94: unconnected-(U1-Pad94) -> /boot0
Routing:
- net VDD: track 61.1 -> 106.7 mm, vias 6 -> 2
- net GND: track 60.6 -> 100.4 mm, vias 3 -> 2
- net /NRST: track 56.0 -> 20.9 mm, vias 0 -> 1
- net /SAI1_FS: track 8.33 -> 29.6 mm, vias 0 -> 1
- net /SPI4_SCK: track 32.3 -> 11.9 mm, vias 2 -> 0
- net /SAI1_SCK: track 6.92 -> 27.2 mm, vias 0 -> 1
- net /SWO: track 24.7 -> 7.76 mm, vias 1 -> 0
- net /SAI1_SD: track 16.5 -> 33.0 mm
- net /SPI1_SCK: track 6.79 -> 21.7 mm
- net /SPI1_MISO: track 7.20 -> 21.6 mm
- net /SWDIO: track 9.51 -> 19.5 mm
- net /SPI4_MOSI: track 26.0 -> 17.0 mm, vias 1 -> 0
- net /SPI3_MISO: track 39.6 -> 30.7 mm, vias 3 -> 0
- net /SPI3_SCK: track 24.8 -> 33.7 mm, vias 3 -> 1
- net /OSC_OUT: track 0.00 -> 7.77 mm
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Other:
- board size 33 x 40.6 mm -> 33 x 41.9 mm

Commit message: pcb_11
Parts:
- removed D1: LED, Diode_SMD:D_0201_0603Metric
- removed R3: 680ohm, Resistor_SMD:R_0201_0603Metric
- added C10: 100nF, Capacitor_SMD:C_0603_1608Metric, B.Cu at (109.7, 113.3)
- added C11: 100nF, Capacitor_SMD:C_0603_1608Metric, B.Cu at (108.2, 116.5)
- added C12: 100nF, Capacitor_SMD:C_0603_1608Metric, F.Cu at (113.7, 125.8)
- added C13: 2.2uF, Resistor_SMD:R_0603_1608Metric, F.Cu at (98.7, 106.5)
- added C14: 2.2uF, Resistor_SMD:R_0603_1608Metric, B.Cu at (99.9, 121.7)
- added C15: 100nF, Capacitor_SMD:C_0603_1608Metric, B.Cu at (113.8, 128.9)
- added C16: 100nF, Capacitor_SMD:C_0603_1608Metric, B.Cu at (113.8, 130.7)
- added C9: 100nF, Resistor_SMD:R_0603_1608Metric, B.Cu at (113.7, 132.2)
- C1: footprint Capacitor_SMD:C_0201_0603Metric -> Capacitor_SMD:C_0603_1608Metric; moved to B.Cu
- C2: footprint Resistor_SMD:R_0201_0603Metric -> Capacitor_SMD:C_0603_1608Metric; moved to B.Cu
- C3, R1, R2: footprint Resistor_SMD:R_0201_0603Metric -> Resistor_SMD:R_0603_1608Metric
- C4, C5, C6: footprint Capacitor_SMD:C_0201_0603Metric -> Capacitor_SMD:C_0603_1608Metric
- C7, C8: value 1pF -> 18pF; footprint Capacitor_SMD:C_0201_0603Metric -> Capacitor_SMD:C_0603_1608Metric
- Y1: value Crystal -> Crystal 16MHz
- moved C2 18.6 mm to (104.5, 110.2), turned to 180 degrees
- moved C1 16.0 mm to (107.6, 110.2), turned to 180 degrees
- moved R1 1.62 mm to (107.1, 127.6)
- moved R2 0.65 mm to (109.8, 127.6)
- moved C6 0.63 mm to (113.7, 132.1)
- moved C7 0.38 mm to (115.0, 121.0)
- moved C8 0.37 mm to (115.0, 111.4)
- moved C3 0.36 mm to (113.7, 127.3)
- moved C5 0.30 mm to (113.7, 130.5)
- moved C4 0.06 mm to (113.7, 128.8)
Connections:
- J1 pad 11: GND -> unconnected-(J1-Pad11)
- U1 pad 100: unconnected-(U1-Pad100) -> VDD
- U1 pad 19: unconnected-(U1-Pad19) -> GND
- U1 pad 20: unconnected-(U1-Pad20) -> VDD
- U1 pad 21: unconnected-(U1-Pad21) -> VDD
- U1 pad 26: unconnected-(U1-Pad26) -> GND
- U1 pad 27: unconnected-(U1-Pad27) -> VDD
- U1 pad 28: GND -> unconnected-(U1-Pad28)
- U1 pad 48: unconnected-(U1-Pad48) -> /VCAP_1
- U1 pad 49: unconnected-(U1-Pad49) -> GND
- U1 pad 50: unconnected-(U1-Pad50) -> VDD
- U1 pad 6: unconnected-(U1-Pad6) -> VDD
- U1 pad 73: unconnected-(U1-Pad73) -> /VCAP_2
- U1 pad 74: unconnected-(U1-Pad74) -> GND
- U1 pad 75: unconnected-(U1-Pad75) -> VDD
- U1 pad 94: /boot0 -> GND
- U1 pad 99: unconnected-(U1-Pad99) -> GND
- U3 pad P1: unconnected-(U3-PadP1) -> GND
Routing:
- net GND: track 100.4 -> 189.6 mm, vias 2 -> 11
- net VDD: track 106.7 -> 166.2 mm, vias 2 -> 6
- net /boot0: track 5.19 -> 0.00 mm, vias 1 -> 0
- net /VCAP_2: track 0.00 -> 4.40 mm, vias 0 -> 1
- net /SPI2_MISO: track 14.0 -> 18.0 mm
- net /SAI1_SD: track 33.0 -> 36.6 mm
- net /VCAP_1: track 0.00 -> 1.97 mm
- net /SPI3_MISO: track 30.7 -> 32.2 mm
- net /I2C1_SCL: track 17.6 -> 16.1 mm
- net /NRST: track 20.9 -> 22.3 mm
- net Net-(D1-Pad2): track 0.97 -> 0.00 mm
- net /SWDIO: track 19.5 -> 20.3 mm
- net /I2C1_SDA: track 18.9 -> 18.3 mm
- added copper zone on B.Cu, net GND
