File: pcb/pcb.kicad_sch (KiCad schematic)
At the start: 11 parts, among them J1 Conn_01x15 Right, J2 Conn_01x15 Left, P1 Conn_01x06, U1 STM32F756VGTx, U2 MP34DT05-A, U3 ISM330DHCX

Commit message: pcb_5
Parts:
- added J3: DIN41612_02x08_AB_EvenPins, Connector_PinSocket_2.54mm:PinSocket_2x08_P2.54mm_Horizontal, symbol Connector:DIN41612_02x08_AB_EvenPins
Connections:
- net GND: now also J3.b2 (Pin_b2)
- net VDD: now also J3.a2 (Pin_a2)
- net SAI1_FS: now reaches U1.3 (PE4)
- net SAI1_FS: now also J3.b16 (Pin_b16)
- net SPI3_MOSI: now reaches U1.36 (PB2)
- net SPI3_MOSI: now also J3.b6 (Pin_b6)
- net SAI1_SCK: now reaches U1.4 (PE5)
- net SAI1_SCK: now also J3.b14 (Pin_b14)
- net SPI4_NSS: now reaches U1.41 (PE11)
- net SPI4_NSS: now also J3.a10 (Pin_a10)
- net SPI4_SCK: now reaches U1.42 (PE12)
- net SPI4_SCK: now also J3.a8 (Pin_a8)
- net SPI4_MISO: now reaches U1.43 (PE13)
- net SPI4_MISO: now also J3.a4 (Pin_a4)
- net SPI4_MOSI: now reaches U1.44 (PE14)
- net SPI4_MOSI: now also J3.a6 (Pin_a6)
- net SAI2_SD: now reaches U1.58 (PD11)
- net SAI2_SD: now also J3.a12 (Pin_a12)
- net SAI2_FS: now reaches U1.59 (PD12)
- net SAI2_FS: now also J3.a16 (Pin_a16)
- net SAI2_SCK: now reaches U1.60 (PD13)
- net SAI2_SCK: now also J3.a14 (Pin_a14)
- net SPI3_NSS: now reaches U1.77 (PA15)
- net SPI3_NSS: now also J3.b10 (Pin_b10)
- net SPI3_SCK: now reaches U1.78 (PC10)
- net SPI3_SCK: now also J3.b8 (Pin_b8)
- net SPI3_MISO: now reaches U1.79 (PC11)
- net SPI3_MISO: now also J3.b4 (Pin_b4)
- net SAI1_SD: now reaches U1.87 (PD6)
- net SAI1_SD: now also J3.b12 (Pin_b12)

Commit message: pcb_6
Parts:
- C1: footprint (none) -> Capacitor_SMD:C_0201_0603Metric
- C2, R1, R2: footprint (none) -> Resistor_SMD:R_0201_0603Metric
- C3: value C -> 100nF; footprint (none) -> Resistor_SMD:R_0201_0603Metric
Connections:
- net GND: now also C1.2, C2.2, J3.2 (Pin_b2), U2.GND; no longer J3.b2 (Pin_b2)
- net SAI1_FS: now also J3.16 (Pin_b16); no longer J3.b16 (Pin_b16)
- net SAI1_SCK: now also J3.14 (Pin_b14); no longer J3.b14 (Pin_b14)
- net SAI1_SD: now also J3.12 (Pin_b12); no longer J3.b12 (Pin_b12)
- net SAI2_FS: now also J3.15 (Pin_a16); no longer J3.a16 (Pin_a16)
- net SAI2_SCK: now also J3.13 (Pin_a14); no longer J3.a14 (Pin_a14)
- net SAI2_SD: now also J3.11 (Pin_a12); no longer J3.a12 (Pin_a12)
- net SPI3_MISO: now also J3.4 (Pin_b4); no longer J3.b4 (Pin_b4)
- net SPI3_MOSI: now also J3.6 (Pin_b6); no longer J3.b6 (Pin_b6)
- net SPI3_NSS: now also J3.10 (Pin_b10); no longer J3.b10 (Pin_b10)
- net SPI3_SCK: now also J3.8 (Pin_b8); no longer J3.b8 (Pin_b8)
- net SPI4_MISO: now also J3.3 (Pin_a4); no longer J3.a4 (Pin_a4)
- net SPI4_MOSI: now also J3.5 (Pin_a6); no longer J3.a6 (Pin_a6)
- net SPI4_NSS: now also J3.9 (Pin_a10); no longer J3.a10 (Pin_a10)
- net SPI4_SCK: now also J3.7 (Pin_a8); no longer J3.a8 (Pin_a8)
- net VDD: now also J3.1 (Pin_a2); no longer J3.a2 (Pin_a2)
Changed lines of the file:
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@@
 (kicad_sch (version 20211123) (generator eeschema)
   (paper "A4")
+  (junction (at 110.49 29.21) (diameter 0) (color 0 0 0 0)
+  )
   (junction (at 133.35 74.93) (diameter 0) (color 0 0 0 0)
   )
@@
     (stroke (width 0) (type default) (color 0 0 0 0))
   )
+  (wire (pts (xy 110.49 29.21) (xy 119.38 29.21))
+    (stroke (width 0) (type default) (color 0 0 0 0))
+  )
   (wire (pts (xy 100.33 38.1) (xy 100.33 39.37))
     (stroke (width 0) (type default) (color 0 0 0 0))
@@
     (stroke (width 0) (type default) (color 0 0 0 0))
   )
-  (wire (pts (xy 100.33 29.21) (xy 119.38 29.21))
+  (wire (pts (xy 100.33 29.21) (xy 110.49 29.21))
     (stroke (width 0) (type default) (color 0 0 0 0))
   )
@@
     (pin "1")
   )
+  (symbol (lib_id "power:GND") (at 110.49 29.21 180) (unit 1)
+    (in_bom yes) (on_board yes) (fields_autoplaced)
+    (property "Reference" "#PWR0117" (id 0) (at 110.49 22.86 0)
+      (effects (font (size 1.27 1.27)) hide)
+    )
+    (property "Value" "GND" (id 1) (at 113.03 27.9399 0)
+      (effects (font (size 1.27 1.27)) (justify right))
+    )
+    (property "Footprint" "" (id 2) (at 110.49 29.21 0)
+      (effects (font (size 1.27 1.27)) hide)
+    )
+    (property "Datasheet" "" (id 3) (at 110.49 29.21 0)
+      (effects (font (size 1.27 1.27)) hide)
+    )
+    (pin "1")
+  )
   (symbol (lib_id "Device:C") (at 133.35 83.82 0) (unit 1)
-    (in_bom yes) (on_board yes) (fields_autoplaced)
-    (property "Reference" "C3" (id 0) (at 137.16 82.5499 0)
-      (effects (font (size 1.27 1.27)) (justify left))
-    )
-    (property "Value" "C" (id 1) (at 137.16 85.0899 0)
-      (effects (font (size 1.27 1.27)) (justify left))
-    )
-    (property "Footprint" "" (id 2) (at 134.3152 87.63 0)
+    (in_bom yes) (on_board yes)
+    (property "Reference" "C3" (id 0) (at 125.73 82.55 0)
+      (effects (font (size 1.27 1.27)) (justify left))
+    )
+    (property "Value" "100nF" (id 1) (at 124.46 85.09 0)
+      (effects (font (size 1.27 1.27)) (justify left))
+    )
+    (property "Footprint" "Resistor_SMD:R_0201_0603Metric" (id 2) (at 134.3152 87.63 0)
       (effects (font (size 1.27 1.27)) hide)
     )
@@
     (property "Reference" "J3" (id 0) (at 120.65 132.08 0))
     (property "Value" "DIN41612_02x08_AB_EvenPins" (id 1) (at 120.65 134.62 0))
-    (property "Footprint" "Connector_PinSocket_2.54mm:PinSocket_2x08_P2.54mm_Horizontal" (id 2) (at 119.38 146.05 0)
-      (effects (font (size 1.27 1.27)) hide)
-    )
+    (property "Footprint" "Connector_PinSocket_2.54mm:PinSocket_2x08_P2.54mm_Horizontal" (id 2) (at 121.92 160.02 0))
     (property "Datasheet" "~" (id 3) (at 119.38 146.05 0)
       (effects (font (size 1.27 1.27)) hide)
     )
-    (pin "a10")
-    (pin "a12")
-    (pin "a14")
-    (pin "a16")
-    (pin "a2")
-    (pin "a4")
-    (pin "a6")
-    (pin "a8")
-    (pin "b10")
-    (pin "b12")
-    (pin "b14")
-    (pin "b16")
-    (pin "b2")
-    (pin "b4")
-    (pin "b6")
-    (pin "b8")
+    (pin "9")
+    (pin "11")
+    (pin "13")
+    (pin "15")
+    (pin "1")
+    (pin "3")
+    (pin "5")
+    (pin "7")
+    (pin "10")
+    (pin "12")
+    (pin "14")
+    (pin "16")
+    (pin "2")
+    (pin "4")
+    (pin "6")
+    (pin "8")
   )
   (symbol (lib_id "Device:R") (at 175.26 68.58 90) (unit 1)
@@
     (property "Reference" "R2" (id 0) (at 175.26 62.23 90))
     (property "Value" "10kOhm" (id 1) (at 175.26 64.77 90))
-    (property "Footprint" "" (id 2) (at 175.26 70.358 90)
+    (property "Footprint" "Resistor_SMD:R_0201_0603Metric" (id 2) (at 175.26 70.358 90)
       (effects (font (size 1.27 1.27)) hide)
     )
@@
       (effects (font (size 1.27 1.27)) (justify right))
     )
-    (property "Footprint" "" (id 2) (at 99.3648 30.48 0)
+    (property "Footprint" "Resistor_SMD:R_0201_0603Metric" (id 2) (at 99.3648 30.48 0)
       (effects (font (size 1.27 1.27)) hide)
     )
@@
       (effects (font (size 1.27 1.27)) (justify right))
     )
-    (property "Footprint" "" (id 2) (at 85.3948 30.48 0)
+    (property "Footprint" "Capacitor_SMD:C_0201_0603Metric" (id 2) (at 85.3948 30.48 0)
       (effects (font (size 1.27 1.27)) hide)
     )
@@
     (property "Reference" "R1" (id 0) (at 175.26 53.34 90))
     (property "Value" "10kOhm" (id 1) (at 175.26 55.88 90))
-    (property "Footprint" "" (id 2) (at 175.26 61.468 90)
+    (property "Footprint" "Resistor_SMD:R_0201_0603Metric" (id 2) (at 175.26 61.468 90)
       (effects (font (size 1.27 1.27)) hide)
     )
@@
       (reference "#PWR0116") (unit 1) (value "VDD") (footprint "")
     )
+    (path "/0d66bee2-895a-43c9-b0a8-f8c61a5e9235"
+      (reference "#PWR0117") (unit 1) (value "GND") (footprint "")
+    )
     (path "/b4ed59f3-175d-4a8b-92bc-fb012e30dd94"
-      (reference "C1") (unit 1) (value "100nF") (footprint "")
+      (reference "C1") (unit 1) (value "100nF") (footprint "Capacitor_SMD:C_0201_0603Metric")
     )
     (path "/6aa487e2-7ef8-49a9-9aa8-7d32950547bb"
-      (reference "C2") (unit 1) (value "1uF") (footprint "")
+      (reference "C2") (unit 1) (value "1uF") (footprint "Resistor_SMD:R_0201_0603Metric")
     )
     (path "/26ba81ac-ef87-41cd-9e57-9e9b3d975584"
-      (reference "C3") (unit 1) (value "C") (footprint "")
+      (reference "C3") (unit 1) (value "100nF") (footprint "Resistor_SMD:R_0201_0603Metric")
     )
     (path "/4d42e9c1-68d4-4062-b21a-69010d8e0318"
@@
     )
     (path "/fced3abb-6c16-461e-8556-b234d8fcefac"
-      (reference "R1") (unit 1) (value "10kOhm") (footprint "")
+      (reference "R1") (unit 1) (value "10kOhm") (footprint "Resistor_SMD:R_0201_0603Metric")
     )
     (path "/473935ce-32f4-4b34-b315-6d773b0ebea7"
-      (reference "R2") (unit 1) (value "10kOhm") (footprint "")
+      (reference "R2") (unit 1) (value "10kOhm") (footprint "Resistor_SMD:R_0201_0603Metric")
     )
     (path "/31b49864-d5c3-4310-8056-1381014dc615"

Commit message: pcb_8
Parts:
- added C4, C5, C6: 100nF, Capacitor_SMD:C_0201_0603Metric, symbol Device:C
- added C7, C8: 1pF, Capacitor_SMD:C_0201_0603Metric, symbol Device:C
- added D1: LED, Diode_SMD:D_0201_0603Metric, symbol Device:LED
- added R3: 680ohm, Resistor_SMD:R_0201_0603Metric, symbol Device:R
- added Y1: Crystal, Crystal:Crystal_SMD_Abracon_ABM3-2Pin_5.0x3.2mm, symbol Device:Crystal
Connections:
- net GND: now also C4.1, C5.1, C6.1, C7.1, C8.1, D1.1 (K)
- net VDD: now also C4.2, C5.2, C6.2
- net OSC_IN: now reaches U1.12 (PH0)
- net OSC_IN: now also C7.2, Y1.1
- net OSC_OUT: now reaches U1.13 (PH1)
- net OSC_OUT: now also C8.2, Y1.2
- net boot0: now reaches U1.94 (BOOT0)
- net boot0: now also R3.2
- new net: D1.2 (A), R3.1
Other:
- moved on the sheet: C1, C2, C3, J3, R1, R2, U2, U3

Commit message: pcb_10
Parts:
- removed D1: LED, Diode_SMD:D_0201_0603Metric, symbol Device:LED
- removed R3: 680ohm, Resistor_SMD:R_0201_0603Metric, symbol Device:R
- added C10, C11, C12: 100nF, Capacitor_SMD:C_0603_1608Metric, symbol Device:C
- added C13, C14: 2.2uF, Resistor_SMD:R_0603_1608Metric, symbol Device:C
- added C9: 100nF, Resistor_SMD:R_0603_1608Metric, symbol Device:C
- C1, C4, C5, C6: footprint Capacitor_SMD:C_0201_0603Metric -> Capacitor_SMD:C_0603_1608Metric
- C2: footprint Resistor_SMD:R_0201_0603Metric -> Capacitor_SMD:C_0603_1608Metric
- C3, R1, R2: footprint Resistor_SMD:R_0201_0603Metric -> Resistor_SMD:R_0603_1608Metric
- C7, C8: value 1pF -> 18pF; footprint Capacitor_SMD:C_0201_0603Metric -> Capacitor_SMD:C_0603_1608Metric
- Y1: value Crystal -> Crystal 16MHz
Connections:
- net boot0 is gone; now on net GND: U1.94 (BOOT0)
- net GND: now also U1.19 (VSSA), U1.26 (VSS), U1.49 (VSS), U1.74 (VSS), U1.99 (VSS), U3.P1 (SDO/SA0), C10.1, C11.1, C12.1, C13.2, C14.2, C9.2; no longer J1.11 (Pin_11), U1.28 (PA4)
- net SPI3_MOSI: now also U1.80 (PC12); no longer U1.36 (PB2)
- net VDD: now also U1.100 (VDD), U1.21 (VDDA), U1.27 (VDD), U1.50 (VDD), U1.75 (VDD), C10.2, C11.2, C12.2, C9.1
- net VCAP_1: now reaches U1.48 (VCAP_1)
- net VCAP_1: now also C13.1
- net VCAP_2: now reaches U1.73 (VCAP_2)
- net VCAP_2: now also C14.1
Other:
- note added: "vdd"
- note added: "vdda"
- note removed: "SPI1_SS"

Commit message: pcb_11
Parts:
- added C15, C16: 100nF, Capacitor_SMD:C_0603_1608Metric, symbol Device:C
Connections:
- net GND: now also C15.1, C16.1
- net SPI3_MOSI: now also U1.36 (PB2); no longer U1.80 (PC12)
- net VDD: now also U1.20 (VREF+), U1.6 (VBAT), C15.2, C16.2
Changed lines of the file:
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@@
   (junction (at 134.62 175.26) (diameter 0) (color 0 0 0 0)
   )
+  (junction (at 120.65 144.78) (diameter 0) (color 0 0 0 0)
+  )
   (junction (at 43.18 179.07) (diameter 0) (color 0 0 0 0)
   )
@@
   (junction (at 182.88 53.34) (diameter 0) (color 0 0 0 0)
   )
+  (junction (at 120.65 132.08) (diameter 0) (color 0 0 0 0)
+  )
   (junction (at 148.59 187.96) (diameter 0) (color 0 0 0 0)
   )
@@
     (stroke (width 0) (type default) (color 0 0 0 0))
   )
+  (wire (pts (xy 120.65 142.24) (xy 120.65 144.78))
+    (stroke (width 0) (type default) (color 0 0 0 0))
+  )
   (wire (pts (xy 163.83 24.13) (xy 163.83 22.86))
     (stroke (width 0) (type default) (color 0 0 0 0))
@@
     (stroke (width 0) (type default) (color 0 0 0 0))
   )
+  (wire (pts (xy 43.18 35.56) (xy 43.18 31.75))
+    (stroke (width 0) (type default) (color 0 0 0 0))
+  )
   (wire (pts (xy 48.26 31.75) (xy 50.8 31.75))
     (stroke (width 0) (type default) (color 0 0 0 0))
@@
     (stroke (width 0) (type default) (color 0 0 0 0))
   )
+  (wire (pts (xy 105.41 134.62) (xy 105.41 132.08))
+    (stroke (width 0) (type default) (color 0 0 0 0))
+  )
   (wire (pts (xy 193.04 62.23) (xy 193.04 71.12))
     (stroke (width 0) (type default) (color 0 0 0 0))
@@
     (stroke (width 0) (type default) (color 0 0 0 0))
   )
+  (wire (pts (xy 43.18 31.75) (xy 45.72 31.75))
+    (stroke (width 0) (type default) (color 0 0 0 0))
+  )
   (wire (pts (xy 119.38 175.26) (xy 119.38 177.8))
     (stroke (width 0) (type default) (color 0 0 0 0))
@@
     (stroke (width 0) (type default) (color 0 0 0 0))
   )
+  (wire (pts (xy 105.41 132.08) (xy 120.65 132.08))
+    (stroke (width 0) (type default) (color 0 0 0 0))
+  )
   (wire (pts (xy 129.54 68.58) (xy 129.54 73.66))
     (stroke (width 0) (type default) (color 0 0 0 0))
@@
     (stroke (width 0) (type default) (color 0 0 0 0))
   )
+  (wire (pts (xy 105.41 144.78) (xy 105.41 142.24))
+    (stroke (width 0) (type default) (color 0 0 0 0))
+  )
   (wire (pts (xy 180.34 78.74) (xy 184.15 78.74))
     (stroke (width 0) (type default) (color 0 0 0 0))
@@
     (stroke (width 0) (type default) (color 0 0 0 0))
   )
+  (wire (pts (xy 120.65 132.08) (xy 120.65 134.62))
+    (stroke (width 0) (type default) (color 0 0 0 0))
+  )
   (wire (pts (xy 163.83 22.86) (xy 149.86 22.86))
     (stroke (width 0) (type default) (color 0 0 0 0))
@@
   )
   (wire (pts (xy 88.9 175.26) (xy 104.14 175.26))
+    (stroke (width 0) (type default) (color 0 0 0 0))
+  )
+  (wire (pts (xy 120.65 144.78) (xy 105.41 144.78))
     (stroke (width 0) (type default) (color 0 0 0 0))
   )
@@
     (effects (font (size 1.27 1.27)) (justify left bottom))
   )
-  (label "SPI3_MOSI" (at 71.12 160.02 0)
+  (label "SPI3_MOSI" (at 71.12 91.44 0)
     (effects (font (size 1.27 1.27)) (justify left bottom))
   )
@@
   (symbol (lib_id "power:GND") (at 97.79 104.14 0) (unit 1)
     (in_bom yes) (on_board yes) (fields_autoplaced)
-    (property "Reference" "#PWR?" (id 0) (at 97.79 110.49 0)
+    (property "Reference" "#PWR0108" (id 0) (at 97.79 110.49 0)
       (effects (font (size 1.27 1.27)) hide)
     )
@@
     )
     (property "Datasheet" "" (id 3) (at 97.79 104.14 0)
+      (effects (font (size 1.27 1.27)) hide)
+    )
+    (pin "1")
+  )
+  (symbol (lib_id "power:VDD") (at 120.65 132.08 0) (unit 1)
+    (in_bom yes) (on_board yes) (fields_autoplaced)
+    (property "Reference" "#PWR0122" (id 0) (at 120.65 135.89 0)
+      (effects (font (size 1.27 1.27)) hide)
+    )
+    (property "Value" "VDD" (id 1) (at 120.65 127 0))
+    (property "Footprint" "" (id 2) (at 120.65 132.08 0)
+      (effects (font (size 1.27 1.27)) hide)
+    )
+    (property "Datasheet" "" (id 3) (at 120.65 132.08 0)
       (effects (font (size 1.27 1.27)) hide)
     )
@@
   (symbol (lib_id "power:GND") (at 129.54 81.28 0) (unit 1)
     (in_bom yes) (on_board yes) (fields_autoplaced)
-    (property "Reference" "#PWR?" (id 0) (at 129.54 87.63 0)
+    (property "Reference" "#PWR0124" (id 0) (at 129.54 87.63 0)
       (effects (font (size 1.27 1.27)) hide)
     )
@@
   (symbol (lib_id "power:GND") (at 113.03 104.14 0) (unit 1)
     (in_bom yes) (on_board yes) (fields_autoplaced)
-    (property "Reference" "#PWR?" (id 0) (at 113.03 110.49 0)
+    (property "Reference" "#PWR0107" (id 0) (at 113.03 110.49 0)
       (effects (font (size 1.27 1.27)) hide)
     )
@@
     (pin "1")
   )
+  (symbol (lib_id "power:GND") (at 120.65 144.78 0) (unit 1)
+    (in_bom yes) (on_board yes) (fields_autoplaced)
+    (property "Reference" "#PWR0126" (id 0) (at 120.65 151.13 0)
+      (effects (font (size 1.27 1.27)) hide)
+    )
+    (property "Value" "GND" (id 1) (at 120.65 149.86 0))
+    (property "Footprint" "" (id 2) (at 120.65 144.78 0)
+      (effects (font (size 1.27 1.27)) hide)
+    )
+    (property "Datasheet" "" (id 3) (at 120.65 144.78 0)
+      (effects (font (size 1.27 1.27)) hide)
+    )
+    (pin "1")
+  )
   (symbol (lib_id "power:VDD") (at 177.8 35.56 180) (unit 1)
     (in_bom yes) (on_board yes) (fields_autoplaced)
@@
     (pin "1")
   )
+  (symbol (lib_id "Device:C") (at 120.65 138.43 180) (unit 1)
+    (in_bom yes) (on_board yes) (fields_autoplaced)
+    (property "Reference" "C16" (id 0) (at 124.46 137.1599 0)
+      (effects (font (size 1.27 1.27)) (justify right))
+    )
+    (property "Value" "100nF" (id 1) (at 124.46 139.6999 0)
+      (effects (font (size 1.27 1.27)) (justify right))
+    )
+    (property "Footprint" "Capacitor_SMD:C_0603_1608Metric" (id 2) (at 119.6848 134.62 0)
+      (effects (font (size 1.27 1.27)) hide)
+    )
+    (property "Datasheet" "~" (id 3) (at 120.65 138.43 0)
+      (effects (font (size 1.27 1.27)) hide)
+    )
+    (pin "1")
+    (pin "2")
+  )
   (symbol (lib_id "Device:C") (at 148.59 181.61 180) (unit 1)
     (in_bom yes) (on_board yes) (fields_autoplaced)
@@
   (symbol (lib_id "power:GND") (at 180.34 76.2 90) (unit 1)
     (in_bom yes) (on_board yes) (fields_autoplaced)
-    (property "Reference" "#PWR?" (id 0) (at 186.69 76.2 0)
+    (property "Reference" "#PWR0123" (id 0) (at 186.69 76.2 0)
       (effects (font (size 1.27 1.27)) hide)
     )
@@
     )
     (pin "1")
+  )
+  (symbol (lib_id "Device:C") (at 105.41 138.43 180) (unit 1)
+    (in_bom yes) (on_board yes) (fields_autoplaced)
+    (property "Reference" "C15" (id 0) (at 109.22 137.1599 0)
+      (effects (font (size 1.27 1.27)) (justify right))
+    )
+    (property "Value" "100nF" (id 1) (at 109.22 139.6999 0)
+      (effects (font (size 1.27 1.27)) (justify right))
+    )
+    (property "Footprint" "Capacitor_SMD:C_0603_1608Metric" (id 2) (at 104.4448 134.62 0)
+      (effects (font (size 1.27 1.27)) hide)
+    )
+    (property "Datasheet" "~" (id 3) (at 105.41 138.43 0)
+      (effects (font (size 1.27 1.27)) hide)
+    )
+    (pin "1")
+    (pin "2")
   )
   (symbol (lib_id "power:VDD") (at 104.14 175.26 0) (unit 1)
@@
     )
     (property "Datasheet" "" (id 3) (at 139.7 90.17 0)
+      (effects (font (size 1.27 1.27)) hide)
+    )
+    (pin "1")
+  )
+  (symbol (lib_id "power:VDD") (at 27.94 58.42 90) (unit 1)
+    (in_bom yes) (on_board yes)
+    (property "Reference" "#PWR0125" (id 0) (at 31.75 58.42 0)
+      (effects (font (size 1.27 1.27)) hide)
+    )
+    (property "Value" "VDD" (id 1) (at 27.94 60.96 90)
+      (effects (font (size 1.27 1.27)) (justify left))
+    )
+    (property "Footprint" "" (id 2) (at 27.94 58.42 0)
+      (effects (font (size 1.27 1.27)) hide)
+    )
+    (property "Datasheet" "" (id 3) (at 27.94 58.42 0)
       (effects (font (size 1.27 1.27)) hide)
     )
@@
       (reference "#PWR0106") (unit 1) (value "VDD") (footprint "")
     )
+    (path "/4a8fd34e-78f3-4be0-a814-a52d0944965e"
+      (reference "#PWR0107") (unit 1) (value "GND") (footprint "")
+    )
+    (path "/2958cb81-4356-408b-b0c0-bb74cb948952"
+      (reference "#PWR0108") (unit 1) (value "GND") (footprint "")
+    )
     (path "/a2e9fa44-79c9-4067-846e-ae22d942b353"
       (reference "#PWR0109") (unit 1) (value "GND") (footprint "")
@@
       (reference "#PWR0121") (unit 1) (value "GND") (footprint "")
     )
-    (path "/2958cb81-4356-408b-b0c0-bb74cb948952"
-      (reference "#PWR?") (unit 1) (value "GND") (footprint "")
+    (path "/2a2be73f-08ac-4dfc-a46a-f839b4113074"
+      (reference "#PWR0122") (unit 1) (value "VDD") (footprint "")
+    )
+    (path "/e55f40cd-435b-42e1-9f5f-e4c8236220e6"
+      (reference "#PWR0123") (unit 1) (value "GND") (footprint "")
     )
     (path "/3594fd94-07da-4717-9ce0-203556271044"
-      (reference "#PWR?") (unit 1) (value "GND") (footprint "")
-    )
-    (path "/4a8fd34e-78f3-4be0-a814-a52d0944965e"
-      (reference "#PWR?") (unit 1) (value "GND") (footprint "")
-    )
-    (path "/e55f40cd-435b-42e1-9f5f-e4c8236220e6"
-      (reference "#PWR?") (unit 1) (value "GND") (footprint "")
+      (reference "#PWR0124") (unit 1) (value "GND") (footprint "")
+    )
+    (path "/f9a301ba-8e22-467c-a4bf-770701a350e1"
+      (reference "#PWR0125") (unit 1) (value "VDD") (footprint "")
+    )
+    (path "/8e417d1c-3cb9-46fd-ba99-6ef1379483b6"
+      (reference "#PWR0126") (unit 1) (value "GND") (footprint "")
     )
     (path "/b4ed59f3-175d-4a8b-92bc-fb012e30dd94"
@@
       (reference "C14") (unit 1) (value "2.2uF") (footprint "Resistor_SMD:R_0603_1608Metric")
     )
+    (path "/ebec24cc-4984-48b0-8ea4-00b8d405b549"
+      (reference "C15") (unit 1) (value "100nF") (footprint "Capacitor_SMD:C_0603_1608Metric")
+    )
+    (path "/da8bf401-5498-474f-a074-cfdbaa1220f1"
+      (reference "C16") (unit 1) (value "100nF") (footprint "Capacitor_SMD:C_0603_1608Metric")
+    )
     (path "/4d42e9c1-68d4-4062-b21a-69010d8e0318"
